File: hdd-driver/hdd-driver.kicad_sch (KiCad schematic)
At the start: 20 parts, among them J1 12V IN, J2 HDD motor contacts, U1 WeAct STM32G474CEU6 Core Board, U2 SimpleFOC Mini v1.0 (DRV8313), U3 MT3608 module, set to 12 V

Commit message: hdd-driver: add current sensing and VR coil input, route the board
Schematic:
- RS1 20 mOhm bus shunt between VM and the new net VM_DRV (SimpleFOC "+",
  C1, C2), read by U4 INA181A2 into I_BUS (PA3).
- RS2/RS3 20 mOhm inline in phases A/B, read by U5/U6 INA240A1 (REF at
  mid-supply) into I_A (PA2) and I_B (PA4). U5's inputs are swapped for
  the layout, so I_A reads with the opposite sign.
- J3 VR coil terminal: 22k series resistor, BAV99 clamp and 470 pF filter
  into PA1 (COMP1_INP / ADC12_IN2), biased by a 10k/10k divider.

PCB: the shunt areas are routed by hand with Kelvin sense legs and the
tracks are locked; the phase tracks reach the spring pads on B.Cu from
below. The remaining signal nets were routed with KiCadRoutingTools and
cleaned up; track ends were re-joined after the final part nudges. DRC
with schematic parity: 0 violations, 0 unconnected. Zones are saved
filled.

README and CLAUDE.md: pin table, power diagram, routing notes.
Parts:
- added C4, C5, C6: 100nF, Capacitor_SMD:C_0603_1608Metric, symbol Device:C
- added C7: 470pF, Capacitor_SMD:C_0603_1608Metric, symbol Device:C
- added C8: 1uF, Capacitor_SMD:C_0603_1608Metric, symbol Device:C
- added D3: BAV99, Package_TO_SOT_SMD:SOT-23, symbol Diode:BAV99
- added J3: VR coil, TerminalBlock_Phoenix:TerminalBlock_Phoenix_MPT-0,5-2-2.54_1x02_P2.54mm_Horizontal, symbol Connector:Screw_Terminal_01x02
- added R6: 22k, Resistor_SMD:R_0603_1608Metric, symbol Device:R
- added R7, R8: 10k, Resistor_SMD:R_0603_1608Metric, symbol Device:R
- added RS1, RS2, RS3: 20m, Resistor_SMD:R_1206_3216Metric, symbol Device:R
- added U4: INA181A2, Package_TO_SOT_SMD:SOT-23-6, symbol Amplifier_Current:INA181
- added U5, U6: INA240A1PW, Package_SO:TSSOP-8_4.4x3mm_P0.65mm, symbol Amplifier_Current:INA240A1PW
Connections:
- net GND: now also C4.2, C5.2, C6.2, C7.2, C8.2, D3.1 (K), R8.2, U4.2 (GND), U4.5 (REF), U5.1 (GND), U5.4 (GND), U5.6 (REF2), U6.1 (GND), U6.4 (GND), U6.6 (REF2)
- net PH_A: now also RS2.2, U5.2 (+); no longer U2.13 (M1)
- net PH_B: now also RS3.2, U6.3 (-); no longer U2.14 (M2)
- net VM: now also RS1.1, U4.3 (+); no longer C1.1, C2.1, U2.11 (VM(+))
- net 3V3: now reaches U1.P2.1 (3V3)
- net 3V3: now also C4.1, C5.1, C6.1, D3.2 (A), R7.1, U4.6 (V+), U5.5 (V+), U5.7 (REF1), U6.5 (V+), U6.7 (REF1)
- net I_BUS: now reaches U1.P2.15 (PA3)
- net I_BUS: now also U4.1
- net I_B: now reaches U1.P2.16 (PA4)
- net I_B: now also U6.8
- net VR_IN: now reaches U1.P2.17 (PA1)
- net VR_IN: now also C7.1, D3.3 (K), R6.2
- net I_A: now reaches U1.P2.18 (PA2)
- net I_A: now also U5.8
- new net PH_A_DRV: RS2.1, U2.13 (M1), U5.3 (-)
- new net PH_B_DRV: RS3.1, U2.14 (M2), U6.2 (+)
- new net VM_DRV: C1.1, C2.1, RS1.2, U2.11 (VM(+)), U4.4 (-)
- new net VR_BIAS: C8.1, J3.2 (Pin_2), R7.2, R8.1
- new net VR_P: J3.1 (Pin_1), R6.1
- no-connect marks 35 -> 30
Other:
- note added: "Current sensing (all outputs to ADC pins; 3V3 from the WeAct board). Shunts: 20 mOhm 1 %, 1206, 0.5 W. RS1 + U4 INA181A2: VM bus current, 1 V/A, 0..3.3 A -> I_BUS = PA3 (ADC1_IN4). RS2/RS3 + U5/U6 INA240A1: inline phase A/B current, 0.4 V/A around 1.65 V, +-4 A -> I_A = PA2 (ADC1_IN3), I_B = PA4 (ADC2_IN17): sample both at once in dual ADC mode. U5 inputs are swapped for layout (IN+ = motor side)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"
- note added: "VR pickup coil (under the disc, 60 pulses/rev): one end at VR_BIAS = VDD/2, the other through R6 and the BAV99 clamp to VR_IN = PA1 (COMP1_INP, ADC12_IN2). COMP1 with DAC3 as threshold and hysteresis -> timer input capture for speed and angle."
